Commit message: Gazebo Fortress | collision fixed

File: src/my_robot_description/urdf/mobile_base.gazebo.xacro (robot description, xacro)
@@ -18,5 +18,5 @@
     </gazebo>
     <!-- handled by ROS2 CONTROL -->
-    <!-- <gazebo>
+    <gazebo>
         <plugin filename="gz-sim-joint-state-publisher-system"
                 name="gz::sim::systems::JointStatePublisher">
@@ -24,4 +24,4 @@
             <joint_name>base_right_wheel_joint</joint_name>
         </plugin>
-    </gazebo> -->
+    </gazebo>
 </robot>

File: src/my_robot_description/urdf/mobile_base.urdf.xacro (robot description, xacro)
@@ -4,4 +4,6 @@
      For more information, please see http://wiki.ros.org/sw_urdf_exporter -->
 <robot xmlns:xacro="http://www.ros.org/wiki/xacro">
+  <xacro:property name="wheel_radius" value="0.035" />
+  <xacro:property name="caster_wheel_radius" value="0.015" />
   <link name="base_footprint" />
   <link name="base_link">
@@ -10,6 +12,8 @@
         xyz="0 0 0"
         rpy="-1.5708 0 -1.5708" />
-      <mass
-        value="0.600820640619417" />
+      <!-- <mass
+        value="0.600820640619417" /> -->
+      <mass
+        value="1.600820640619417" />
       <inertia
         ixx="0.00079861144929563"
@@ -57,4 +61,6 @@
         xyz="6.9389E-18 0.0047803 4.1273E-18"
         rpy="1.5708 0 1.5708" /> -->
+      <!-- <mass
+        value="0.0065128" /> -->
       <mass
         value="0.0065128" />
@@ -85,7 +91,10 @@
         xyz="0 0 0"
         rpy="1.5708 0 1.5708" />
-      <geometry>
+      <!-- <geometry>
         <mesh
           filename="package://my_robot_description/meshes/caster_wheel_link.STL" />
+      </geometry> -->
+      <geometry>
+          <sphere radius="${caster_wheel_radius}" />
       </geometry>
     </collision>
@@ -135,7 +144,10 @@
         xyz="0 0 0"
         rpy="0 0 0" />
-      <geometry>
+      <!-- <geometry>
         <mesh
           filename="package://my_robot_description/meshes/right_wheel_link.STL" />
+      </geometry> -->
+      <geometry>
+          <sphere radius="${wheel_radius}" />
       </geometry>
     </collision>
@@ -185,7 +197,10 @@
         xyz="0 0 0"
         rpy="0 0 0" />
-      <geometry>
+      <!-- <geometry>
         <mesh
           filename="package://my_robot_description/meshes/left_wheel_link.STL" />
+      </geometry> -->
+      <geometry>
+          <sphere radius="${wheel_radius}" />
       </geometry>
     </collision>
