Commit message: Gazebo & mapping final

File: src/my_robot_description/urdf/lidar.urdf.xacro (robot description, xacro)
@@ -7,8 +7,12 @@
         </plugin>
     </gazebo>
+    <gazebo reference='base_lidar_joint'>
+        <preserveFixedJoint>true</preserveFixedJoint>
+    </gazebo>
     <gazebo reference='lidar_link'>
         <sensor name='gpu_lidar' type='gpu_lidar'>
             <pose>0 0 0 0 0 0</pose>
             <frame_id>lidar_link</frame_id>
+            <gz_frame_id>lidar_link</gz_frame_id>
             <update_rate>10</update_rate>
             <lidar>
@@ -17,10 +21,10 @@
                         <samples>640</samples>
                         <resolution>1</resolution>
-                        <min_angle>-1.396263</min_angle>
-                        <max_angle>1.396263</max_angle>
+                        <min_angle>-3.1459</min_angle>
+                        <max_angle>3.1459</max_angle>
                     </horizontal>
                     <vertical>
-                        <samples>1</samples>
-                        <resolution>0.01</resolution>
+                        <samples>16</samples>
+                        <resolution>1</resolution>
                         <min_angle>0</min_angle>
                         <max_angle>0</max_angle>
@@ -32,4 +36,9 @@
                     <resolution>0.01</resolution>
                 </range>
+                <noise>
+                    <type>gaussian</type>
+                    <mean>0</mean>
+                    <stddev>0.01</stddev>
+                </noise>
             </lidar>
             <always_on>1</always_on>

File: src/my_robot_description/urdf/mobile_base.urdf.xacro (robot description, xacro)
@@ -225,13 +225,6 @@
         xyz="0 0 0"
         rpy="1.5708 0 0" />
-      <mass
-        value="0.0" />
-      <inertia
-        ixx="0"
-        ixy="0"
-        ixz="0"
-        iyy="0"
-        iyz="0"
-        izz="0" />
+      <mass value="0.01" />
+      <inertia ixx="1e-5" ixy="0" ixz="0" iyy="1e-5" iyz="0" izz="1e-5" />
     </inertial>
     <visual>
@@ -262,5 +255,5 @@
     <origin
       xyz="3E-05 2.5E-05 0.20108"
-      rpy="0 0 3.1416" />
+      rpy="0 0 0" />
       <!-- rpy="1.5708 0 1.5708" /> -->
     <parent
