Commit message: Waypoints added

File: src/my_robot_description/urdf/mobile_base.urdf.xacro (robot description, xacro)
@@ -264,3 +264,45 @@
       xyz="0 0 0" />
   </joint>
+  <link name="imu_link"/>
+  <joint name="imu_joint" type="fixed">
+    <parent link="base_link"/>
+    <child link="imu_link"/>
+    <origin xyz="0.0 0.0 0.0" rpy="0.0 0.0 0.0"/>
+  </joint>
+  <link
+    name="camera_link">
+    <inertial>
+      <origin
+        xyz="1 0 0"
+        rpy="1.5708 0 0" />
+      <mass value="0.01" />
+      <inertia ixx="1e-5" ixy="0" ixz="0" iyy="1e-5" iyz="0" izz="1e-5" />
+    </inertial>
+    <visual>
+      <origin
+        xyz="1 0 0"
+        rpy="1.5708 0 0" />
+      <geometry>
+        <box size="0.6 0.1 0.2"/>
+      </geometry>
+      <material
+        name="">
+        <color
+          rgba="1 1 1 1" />
+      </material>
+    </visual>
+    <collision>
+      <origin
+        xyz="0 0 0"
+        rpy="1.5708 0 0" />
+      <geometry>
+        <box size="0.6 0.1 0.2"/>
+      </geometry>
+    </collision>
+  </link>
+  <joint name="camera_joint" type="fixed">
+    <parent link="lidar_link"/>
+    <child link ="camera_link"/>
+    <origin xyz="0.0 0.0 0.0" rpy="0.0 0.0 0.0"/>
+  </joint>
 </robot>

File: src/my_robot_description/urdf/my_robot.urdf.xacro (robot description, xacro)
@@ -14,3 +14,4 @@
         baud="$(arg baud)" />
     <xacro:include filename="lidar.urdf.xacro" />
+    <xacro:include filename="imu.urdf.xacro" />
 </robot>

Commit message: Slam toolbox config

File: src/my_robot_description/urdf/mobile_base.urdf.xacro (robot description, xacro)
@@ -270,5 +270,5 @@
     <origin xyz="0.0 0.0 0.0" rpy="0.0 0.0 0.0"/>
   </joint>
-  <link
+  <!-- <link
     name="camera_link">
     <inertial>
@@ -300,9 +300,9 @@
       </geometry>
     </collision>
-  </link>
-  <joint name="camera_joint" type="fixed">
+  </link> -->
+  <!-- <joint name="camera_joint" type="fixed">
     <parent link="lidar_link"/>
     <child link ="camera_link"/>
     <origin xyz="0.0 0.0 0.0" rpy="0.0 0.0 0.0"/>
-  </joint>
+  </joint> -->
 </robot>
