Commit message: Fix lidar frame

File: src/my_robot_description/urdf/mobile_base.ros2_control.xacro (robot description, xacro)
@@ -12,5 +12,5 @@
                 <param name="baud">${baud}</param>
                 <param name="timeout_ms">20</param>
-                <param name="counts_per_rev">112.5</param>
+                <param name="counts_per_rev">449</param>
                 <!-- <param name="invert_left">true</param>
                 <param name="invert_right">true</param> -->
@@ -19,5 +19,5 @@
                 <param name="invert_left_enc">false</param>
                 <param name="invert_right_enc">false</param>
-                <param name="max_rad_s">5.0</param>
+                <param name="max_rad_s">20.0</param>
             </hardware>
             </xacro:unless>

File: src/my_robot_description/urdf/mobile_base.urdf.xacro (robot description, xacro)
@@ -25,4 +25,7 @@
     </inertial>
     <visual>
+      <!-- <origin
+        xyz="0 0 0"
+        rpy="0 0 -1.5708" /> -->
       <origin
         xyz="0 0 0"
@@ -255,5 +258,5 @@
     <origin
       xyz="3E-05 2.5E-05 0.20108"
-      rpy="0 0 0" />
+      rpy="0 0 3.14159" />
       <!-- rpy="1.5708 0 1.5708" /> -->
     <parent
